File: Automatic Load Switchover.kicad_sch (KiCad schematic)
At the start: 22 parts, among them Q7 2SJ174, Q8 2SJ174, U13 LTC2952, U14 AMS1117-3.3, U15 LM7805_TO220

Commit message: Final: small edit on silkscreen + BOM file + generating Gerber file.
Parts:
- R36, R40, R41: LINK https://makerselectronics.com/product/chip-resistor-smd-10k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 -> https://makerselectronics.com/product/chip-resistor-smd-1kω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
